Commit message: added meshes for mount and sensor

File: description/urdf/nanoscan3.urdf.xacro (robot description, xacro)
@@ -8,5 +8,4 @@
   <xacro:arg name="sim_gazebo" default="false" />
   <xacro:arg name="simulation_controllers" default="" />
-  <xacro:include filename="$(find sick_safetyscanners2)/description/urdf/nanoscan3/nanoscan3_macro.xacro"/>
   <xacro:include filename="$(find sick_safetyscanners2)/description/urdf/nanoscan3/nanoscan3_macro.ros2_control.xacro"/>
   <!-- create link fixed to the "world" -->
@@ -14,6 +13,11 @@
   <!-- Load robot's macro with parameters -->
   <!-- set prefix if multiple robots are used -->
-  <xacro:nanoscan3 prefix="$(arg prefix)" parent="world" >
-    <origin xyz="0 0 0" rpy="0 0 0" />          <!-- position robot in the world -->
+  <xacro:include filename="$(find sick_safetyscanners2)/description/urdf/nanoscan3/nanoscan3_macro.xacro"/>
+  <xacro:nanoscan3
+    prefix="$(arg prefix)"
+    name="nanoscan3"
+    parent="world"
+    mounting_kit="true">
+    <origin xyz="0 0 0" rpy="0 0 0" />
   </xacro:nanoscan3>
   <xacro:nanoscan3_ros2_control

File: description/urdf/nanoscan3/nanoscan3_macro.xacro (robot description, xacro)
@@ -2,160 +2,14 @@
 <robot xmlns:xacro="http://wiki.ros.org/xacro">
   <xacro:include filename="$(find sick_safetyscanners2)/description/urdf/common.xacro" />
-  <xacro:macro name="nanoscan3" params="prefix parent *origin">
-    <!-- LINKS -->
-    <!-- base link -->
-    <link name="${prefix}base_link">
-      <!-- Default inertial for Gazebo - copy and edit block from 'common.xacro'
-           to get more realistic behavior -->
-      <xacro:default_inertial/>
+  <xacro:macro name="nanoscan3" params="prefix name parent *origin mounting_kit">
+    <link name="${prefix}base_link"/>
+    <link name="${name}">
       <visual>
-        <origin xyz="0 0 0" rpy="0 0 0" />
+        <origin rpy="0 0 0" xyz="0 0 0"/>
         <geometry>
-          <cylinder length="0.3" radius="0.3" />
-<!--           <mesh filename="package://sick_safetyscanners2/meshes/nanoscan3/visual/base_link.dae" /> -->
+          <mesh filename="package://sick_safetyscanners2/description/meshes/nanoscan3/visual/nanoscan3.dae"/>
         </geometry>
       </visual>
-      <collision>
-        <origin xyz="0 0 0" rpy="0 0 0" />
-        <geometry>
-          <cylinder length="0.3" radius="0.3" />
-<!--           <mesh filename="package://sick_safetyscanners2/meshes/nanoscan3/collision/base_link.stl" /> -->
-        </geometry>
-      </collision>
     </link>
-    <!-- link 1 -->
-    <link name="${prefix}link1">
-      <!-- Default inertial for Gazebo - copy and edit block from 'common.xacro'
-           to get more realistic behavior -->
-      <xacro:default_inertial/>
-      <visual>
-        <origin xyz="0 0 0" rpy="0 0 0" />
-        <geometry>
-          <cylinder length="0.3" radius="0.15" />
-<!--           <mesh filename="package://sick_safetyscanners2/meshes/nanoscan3/visual/link1.dae" /> -->
-        </geometry>
-      </visual>
-      <collision>
-        <origin xyz="0 0 0" rpy="0 0 0" />
-        <geometry>
-          <cylinder length="0.3" radius="0.15" />
-<!--           <mesh filename="package://sick_safetyscanners2/meshes/nanoscan3/collision/link1.stl" /> -->
-        </geometry>
-      </collision>
-    </link>
-    <!-- link 2 -->
-    <link name="${prefix}link2">
-      <!-- Default inertial for Gazebo - copy and edit block from 'common.xacro'
-           to get more realistic behavior-->
-      <xacro:default_inertial/>
-      <visual>
-        <origin xyz="0 0 0" rpy="0 0 0" />
-        <geometry>
-          <cylinder length="0.8" radius="0.15" />
-<!--           <mesh filename="package://sick_safetyscanners2/meshes/nanoscan3/visual/link2.dae" /> -->
-        </geometry>
-      </visual>
-      <collision>
-        <origin xyz="0 0 0" rpy="0 0 0" />
-        <geometry>
-          <cylinder length="0.8" radius="0.15" />
-<!--           <mesh filename="package://sick_safetyscanners2/meshes/nanoscan3/collision/link2.stl"  /> -->
-        </geometry>
-      </collision>
-    </link>
-    <!-- link 3 -->
-    <link name="${prefix}link3">
-      <!-- Default inertial for Gazebo - copy and edit block from 'common.xacro'
-           to get more realistic behavior-->
-      <xacro:default_inertial/>
-      <visual>
-        <origin xyz="0 0 0" rpy="0 0 0" />
-        <geometry>
-          <cylinder length="0.5" radius="0.10" />
-<!--           <mesh filename="package://sick_safetyscanners2/meshes/nanoscan3/visual/link3.dae" /> -->
-        </geometry>
-      </visual>
-      <collision>
-        <origin xyz="0 0 0" rpy="0 0 0" />
-        <geometry>
-          <cylinder length="0.5" radius="0.10" />
-<!--           <mesh filename="package://sick_safetyscanners2/meshes/nanoscan3/collision/link3.stl"  /> -->
-        </geometry>
-      </collision>
-    </link>
-    <!-- link 4 -->
-    <link name="${prefix}link4">
-      <!-- Default inertial for Gazebo - copy and edit block from 'common.xacro'
-           to get more realistic behavior-->
-      <xacro:default_inertial/>
-      <visual>
-        <origin xyz="0 0 0" rpy="0 0 0" />
-        <geometry>
-          <cylinder length="0.1" radius="0.2" />
-<!--           <mesh filename="package://sick_safetyscanners2/meshes/nanoscan3/visual/link4.dae" /> -->
-        </geometry>
-      </visual>
-      <collision>
-        <origin xyz="0 0 0" rpy="0 0 0" />
-        <geometry>
-          <cylinder length="0.1" radius="0.2" />
-<!--           <mesh filename="package://sick_safetyscanners2/meshes/nanoscan3/collision/link4.stl"  /> -->
-        </geometry>
-      </collision>
-    </link>
-    <!-- link 5 -->
-    <link name="${prefix}link5">
-      <!-- Default inertial for Gazebo - copy and edit block from 'common.xacro'
-           to get more realistic behavior-->
-      <xacro:default_inertial/>
-      <visual>
-        <origin xyz="0 0 0" rpy="0 0 0" />
-        <geometry>
-          <cylinder length="0.2" radius="0.1" />
-<!--           <mesh filename="package://sick_safetyscanners2/meshes/nanoscan3/visual/link5.dae" /> -->
-        </geometry>
-      </visual>
-      <collision>
-        <origin xyz="0 0 0" rpy="0 0 0" />
-        <geometry>
-          <cylinder length="0.2" radius="0.1" />
-<!--           <mesh filename="package://sick_safetyscanners2/meshes/nanoscan3/collision/link5.stl" /> -->
-        </geometry>
-      </collision>
-    </link>
-    <!-- link 6 -->
-    <link name="${prefix}link6">
-      <!-- Default inertial for Gazebo - copy and edit block from 'common.xacro'
-           to get more realistic behavior-->
-      <xacro:default_inertial/>
-      <visual>
-        <origin xyz="0 0 0" rpy="0 0 0" />
-        <geometry>
-          <cylinder length="0.05" radius="0.1" />
-<!--           <mesh filename="package://sick_safetyscanners2/meshes/nanoscan3/visual/link6.dae" /> -->
-        </geometry>
-      </visual>
-      <collision>
-        <origin xyz="0 0 0" rpy="0 0 0" />
-        <geometry>
-          <cylinder length="0.05" radius="0.1" />
-<!--           <mesh filename="package://sick_safetyscanners2/meshes/nanoscan3/collision/link6.stl" /> -->
-        </geometry>
-      </collision>
-    </link>
-    <!-- All-zero tool frame. This frame should correspond to the TOOL frame of the robot's controller.) -->
-    <link name="${prefix}tool0" />
-    <!-- tool link -->
-<!-- START Delete if not needed -->
-    <!-- Standard frames for industrial robots. Also useful for manipulators.
-         (ROS-I specs - https://wiki.ros.org/Industrial/Tutorials/WorkingWithRosIndustrialRobotSupportPackages#Standardised_links_.2F_frames)-->
-    <!-- This frame should correspond to the BASE coordinate system of robot's controller.) -->
-    <link name="${prefix}base" />
-    <!-- Frame for mounting EEF models to a manipulator. x+ axis points forward (REP 103). -->
-    <link name="${prefix}flange" />
-<!-- END Delete if not needed  -->
-    <!-- END LINKS -->
-    <!-- JOINTS -->
-    <!-- base_joint fixes base_link to the environment -->
     <joint name="${prefix}base_joint" type="fixed">
       <xacro:insert_block name="origin" />
@@ -163,73 +17,9 @@
       <child link="${prefix}base_link" />
     </joint>
-    <!-- joint 1 -->
-    <joint name="${prefix}joint1" type="revolute">
-      <origin xyz="0 0 0.3" rpy="${pi} 0 0" />
+    <joint name="${name}_joint" type="fixed">
       <parent link="${prefix}base_link" />
-      <child link="${prefix}link1" />
-      <axis xyz="0 0 1" />
-      <limit effort="0" lower="${radians(-180)}" upper="${radians(180)}" velocity="${radians(180)}" />
+      <child link="${name}" />
+      <origin rpy="0 0 0" xyz="0 0 0"/>
     </joint>
-    <!-- joint 2 -->
-    <joint name="${prefix}joint2" type="revolute">
-      <origin xyz="0 0 0.3" rpy="${pi/2} 0 0" />
-      <parent link="${prefix}link1" />
-      <child link="${prefix}link2" />
-      <axis xyz="0 0 1" />
-      <limit effort="0" lower="${radians(-180)}" upper="${radians(180)}" velocity="${radians(180)}" />
-    </joint>
-    <!-- joint 3 -->
-    <joint name="${prefix}joint3" type="revolute">
-      <origin xyz="0.8 0 0" rpy="0 0 0" />
-      <parent link="${prefix}link2" />
-      <child link="${prefix}link3" />
-      <axis xyz="0 0 1" />
-      <limit effort="0" lower="${radians(-90)}" upper="${radians(180)}" velocity="${radians(270)}" />
-    </joint>
-    <!-- joint 4 -->
-    <joint name="${prefix}joint4" type="revolute">
-      <origin xyz="0 0.1 0" rpy="0 ${-pi/2} 0" />
-      <parent link="${prefix}link3" />
-      <child link="${prefix}link4" />
-      <axis xyz="0 0 1" />
-      <limit effort="0" lower="${radians(-360)}" upper="${radians(360)}" velocity="${radians(360)}" />
-    </joint>
-    <!-- joint 5 -->
-    <joint name="${prefix}joint5" type="revolute">
-      <origin xyz="0 0 -0.1" rpy="0 ${pi/2} 0" />
-      <parent link="${prefix}link4" />
-      <child link="${prefix}link5" />
-      <axis xyz="0 0 1" />
-      <limit effort="0" lower="${radians(-120)}" upper="${radians(120)}" velocity="${radians(540)}" />
-    </joint>
-    <!-- joint 6 -->
-    <joint name="${prefix}joint6" type="revolute">
-      <origin xyz="0 0 0.1" rpy="0 ${-pi/2} 0" />
-      <parent link="${prefix}link5" />
-      <child link="${prefix}link6" />
-      <axis xyz="0 0 1" />
-      <limit effort="0" lower="${radians(-360)}" upper="${radians(360)}" velocity="${radians(720)}" />
-    </joint>
-    <!-- tool frame - fixed frame -->
-    <joint name="${prefix}joint6-tool0" type="fixed">
-      <parent link="${prefix}link6" />
-      <child link="${prefix}tool0" />
-      <origin xyz="0 0 -0.115" rpy="0 ${-pi} ${-pi/2}" />
-    </joint>
-    <!-- END JOINTS -->
-<!-- START Delete if not needed -->
-    <!-- Standard frames for industrial robots. Also useful for manipulators.
-         (ROS-I specs - https://wiki.ros.org/Industrial/Tutorials/WorkingWithRosIndustrialRobotSupportPackages#Standardised_links_.2F_frames)-->
-    <joint name="${prefix}base_link-base_joint" type="fixed">
-      <origin xyz="0 0 0" rpy="0 0 0" />
-      <parent link="${prefix}base_link" />
-      <child link="${prefix}base" />
-    </joint>
-    <joint name="${prefix}tool0-flange_joint" type="fixed">
-      <origin xyz="0 0 0" rpy="0 0 0" />
-      <parent link="${prefix}tool0" />
-      <child link="${prefix}flange" />
-    </joint>
-<!-- END Delete if not needed  -->
   </xacro:macro>
 </robot>

Commit message: added a "mounting kit" conditional

File: description/urdf/nanoscan3.urdf.xacro (robot description, xacro)
@@ -3,4 +3,5 @@
   <!-- Use this if parameters are set from the launch file, otherwise delete -->
   <xacro:arg name="prefix" default="" />
+  <xacro:arg name="mounting_kit" default="true" />
   <xacro:arg name="use_mock_hardware" default="false" />
   <xacro:arg name="mock_sensor_commands" default="false" />
@@ -14,9 +15,10 @@
   <!-- set prefix if multiple robots are used -->
   <xacro:include filename="$(find sick_safetyscanners2)/description/urdf/nanoscan3/nanoscan3_macro.xacro"/>
+  <xacro:property name="mounting_kit" value="$(arg mounting_kit)"/>
   <xacro:nanoscan3
     prefix="$(arg prefix)"
     name="nanoscan3"
     parent="world"
-    mounting_kit="true">
+    mounting_kit="${mounting_kit}">
     <origin xyz="0 0 0" rpy="0 0 0" />
   </xacro:nanoscan3>

File: description/urdf/nanoscan3/nanoscan3_macro.xacro (robot description, xacro)
@@ -9,24 +9,34 @@
   <xacro:property name="sensor_rot_z" value="${radians(-90)}"/>
   <xacro:macro name="nanoscan3" params="prefix name parent *origin mounting_kit">
-  <!-- MOUNT -->
-    <joint name="${prefix}${name}_mount_joint" type="fixed">
-      <xacro:insert_block name="origin" />
-      <parent link="${parent}" />
-      <child link="${prefix}${name}_mount" />
-    </joint>
-    <link name="${prefix}${name}_mount">
-      <visual>
+    <xacro:if value="${mounting_kit}">
+      <!-- MOUNT -->
+      <joint name="${prefix}${name}_mount_joint" type="fixed">
         <xacro:insert_block name="origin" />
-        <geometry>
-          <mesh filename="package://sick_safetyscanners2/description/meshes/nanoscan3/visual/mount.dae"/>
-        </geometry>
-      </visual>
-    </link>
-  <!-- SENSOR BASE -->
-    <joint name="${prefix}${name}_base_joint" type="fixed">
-      <origin xyz="${base_x} ${base_y} 0"/>
-      <parent link="${prefix}${name}_mount" />
-      <child link="${prefix}${name}_base" />
-    </joint>
+        <parent link="${parent}" />
+        <child link="${prefix}${name}_mount" />
+      </joint>
+      <link name="${prefix}${name}_mount">
+        <visual>
+          <xacro:insert_block name="origin" />
+          <geometry>
+            <mesh filename="package://sick_safetyscanners2/description/meshes/nanoscan3/visual/mount.dae"/>
+          </geometry>
+        </visual>
+      </link>
+      <!-- SENSOR BASE when mounted -->
+      <joint name="${prefix}${name}_base_joint" type="fixed">
+        <origin xyz="${base_x} ${base_y} 0"/>
+        <parent link="${prefix}${name}_mount" />
+        <child link="${prefix}${name}_base" />
+      </joint>
+    </xacro:if>
+    <xacro:unless value="${mounting_kit}">
+      <!-- SENSOR BASE without mount-->
+      <joint name="${prefix}${name}_base_joint" type="fixed">
+        <xacro:insert_block name="origin" />
+        <parent link="${parent}" />
+        <child link="${prefix}${name}_base" />
+      </joint>
+    </xacro:unless>
     <link name="${prefix}${name}_base">
       <origin xyz="${-base_x} ${-base_y} 0"/>

Commit message: removed unecessary, adjusted origin, colored MountingKit

File: description/urdf/nanoscan3.urdf.xacro (robot description, xacro)
@@ -2,12 +2,6 @@
 <robot xmlns:xacro="http://wiki.ros.org/xacro" name="nanoscan3">
   <!-- Use this if parameters are set from the launch file, otherwise delete -->
-  <xacro:arg name="prefix" default="" />
   <xacro:arg name="mounting_kit" default="true" />
-  <xacro:arg name="use_mock_hardware" default="false" />
-  <xacro:arg name="mock_sensor_commands" default="false" />
-  <xacro:arg name="sim_gazebo_classic" default="false" />
   <xacro:arg name="sim_gazebo" default="false" />
-  <xacro:arg name="simulation_controllers" default="" />
-  <xacro:include filename="$(find sick_safetyscanners2)/description/urdf/nanoscan3/nanoscan3_macro.ros2_control.xacro"/>
   <!-- create link fixed to the "world" -->
   <link name="world" />
@@ -17,5 +11,4 @@
   <xacro:property name="mounting_kit" value="$(arg mounting_kit)"/>
   <xacro:nanoscan3
-    prefix="$(arg prefix)"
     name="nanoscan3"
     parent="world"
@@ -23,11 +16,3 @@
     <origin xyz="0 0 0" rpy="0 0 0" />
   </xacro:nanoscan3>
-  <xacro:nanoscan3_ros2_control
-    name="nanoscan3"
-    prefix="$(arg prefix)"
-    use_mock_hardware="$(arg use_mock_hardware)"
-    mock_sensor_commands="$(arg mock_sensor_commands)"
-    sim_gazebo_classic="$(arg sim_gazebo_classic)"
-    sim_gazebo="$(arg sim_gazebo)"
-    simulation_controllers="$(arg simulation_controllers)" />
 </robot>

File: description/urdf/nanoscan3/nanoscan3_macro.xacro (robot description, xacro)
@@ -8,18 +8,17 @@
   <xacro:property name="sensor_z" value="0.0315"/>
   <xacro:property name="sensor_rot_z" value="${radians(-90)}"/>
-  <xacro:macro name="nanoscan3" params="prefix name parent *origin mounting_kit">
+  <xacro:macro name="nanoscan3" params="name parent *origin mounting_kit">
     <xacro:if value="${mounting_kit}">
       <!-- MOUNT -->
-      <joint name="${prefix}${name}_mount_joint" type="fixed">
+      <joint name="${name}_mount_joint" type="fixed">
         <xacro:insert_block name="origin" />
         <parent link="${parent}" />
-        <child link="${prefix}${name}_mount" />
+        <child link="${name}_mount" />
       </joint>
-      <link name="${prefix}${name}_mount">
+      <link name="${name}_mount">
         <!-- Default inertial for Gazebo - copy and edit block from 'common.xacro'
             to get more realistic behavior -->
         <xacro:default_inertial/>
         <visual>
-          <xacro:insert_block name="origin" />
           <geometry>
             <mesh filename="package://sick_safetyscanners2/description/meshes/MountingKit_2a.dae"/>
@@ -27,5 +26,4 @@
         </visual>
         <collision>
-          <xacro:insert_block name="origin" />
           <geometry>
             <mesh filename="package://sick_safetyscanners2/description/meshes/MountingKit_2a_collision.stl"/>
@@ -34,28 +32,28 @@
       </link>
       <!-- SENSOR BASE when mounted -->
-      <joint name="${prefix}${name}_base_joint" type="fixed">
+      <joint name="${name}_base_joint" type="fixed">
         <origin xyz="${base_x} ${base_y} 0"/>
-        <parent link="${prefix}${name}_mount" />
-        <child link="${prefix}${name}_base" />
+        <parent link="${name}_mount" />
+        <child link="${name}_base" />
       </joint>
     </xacro:if>
     <xacro:unless value="${mounting_kit}">
       <!-- SENSOR BASE without mount-->
-      <joint name="${prefix}${name}_base_joint" type="fixed">
+      <joint name="${name}_base_joint" type="fixed">
         <xacro:insert_block name="origin" />
         <parent link="${parent}" />
-        <child link="${prefix}${name}_base" />
+        <child link="${name}_base" />
       </joint>
     </xacro:unless>
-    <link name="${prefix}${name}_base">
+    <link name="${name}_base">
       <origin xyz="${-base_x} ${-base_y} 0"/>
     </link>
   <!-- SENSOR FRAME -->
     <joint name="${name}_joint" type="fixed">
-      <parent link="${prefix}${name}_base" />
-      <child link="${prefix}${name}" />
+      <parent link="${name}_base" />
+      <child link="${name}" />
       <origin xyz="0 ${sensor_y} ${sensor_z}" rpy="0 0 ${sensor_rot_z}"/>
     </joint>
-    <link name="${prefix}${name}">
+    <link name="${name}">
       <!-- Default inertial for Gazebo - copy and edit block from 'common.xacro'
            to get more realistic behavior -->

Commit message: enabled gazebo integration in urdf

File: description/urdf/nanoscan3.urdf.xacro (robot description, xacro)
@@ -13,5 +13,13 @@
     name="nanoscan3"
     parent="world"
-    mounting_kit="${mounting_kit}">
+    mounting_kit="${mounting_kit}"
+    ros_topic="/nanoscan3_topic"
+    update_rate="50.0"
+    min_angle="${radians(-45)}"
+    max_angle="${radians(225)}"
+    min_range="0.05"
+    max_range="10.0"
+    gaussian_noise="0.006"
+    max_beams="500">
     <origin xyz="0 0 0" rpy="0 0 0" />
   </xacro:nanoscan3>

File: description/urdf/nanoscan3/nanoscan3_macro.xacro (robot description, xacro)
@@ -2,4 +2,5 @@
 <robot xmlns:xacro="http://wiki.ros.org/xacro">
   <xacro:include filename="$(find sick_safetyscanners2)/description/urdf/common.xacro" />
+  <xacro:include filename="$(find sick_safetyscanners2)/description/urdf/nanoscan3/gazebo_macro.xacro" />
   <!-- joint offsets when mounted on frame -->
   <xacro:property name="base_x" value="0.0803"/>
@@ -8,5 +9,19 @@
   <xacro:property name="sensor_z" value="0.0315"/>
   <xacro:property name="sensor_rot_z" value="${radians(-90)}"/>
-  <xacro:macro name="nanoscan3" params="name parent *origin mounting_kit">
+  <xacro:macro name="nanoscan3"
+    params="
+      name
+      parent
+      mounting_kit
+      ros_topic
+      update_rate
+      min_angle
+      max_angle
+      min_range
+      max_range
+      gaussian_noise:=0.006
+      max_beams:=540
+      *origin
+    ">
     <xacro:if value="${mounting_kit}">
       <!-- MOUNT -->
@@ -72,4 +87,17 @@
       </collision>
     </link>
+    <!-- gazebo integration -->
+    <xacro:sick_safetyscanners2_gazebo
+      name="${name}"
+      link="${name}"
+      ros_topic="${ros_topic}"
+      update_rate="${update_rate}"
+      min_angle="${min_angle}"
+      max_angle="${max_angle}"
+      min_range="${min_range}"
+      max_range="${max_range}"
+      gaussian_noise="${gaussian_noise}"
+      max_beams="${max_beams}">
+    </xacro:sick_safetyscanners2_gazebo>
   </xacro:macro>
 </robot>
