Commit message: adjusted joint origins

File: description/urdf/nanoscan3/nanoscan3_macro.xacro (robot description, xacro)
@@ -2,9 +2,43 @@
 <robot xmlns:xacro="http://wiki.ros.org/xacro">
   <xacro:include filename="$(find sick_safetyscanners2)/description/urdf/common.xacro" />
+  <!-- joint offsets when mounted on frame -->
+  <xacro:property name="base_x" value="0.0803"/>
+  <xacro:property name="base_y" value="-0.053"/>
+  <xacro:property name="sensor_y" value="${-base_y}"/>
+  <xacro:property name="sensor_z" value="0.0315"/>
+  <xacro:property name="sensor_rot_z" value="${radians(-90)}"/>
   <xacro:macro name="nanoscan3" params="prefix name parent *origin mounting_kit">
-    <link name="${prefix}base_link"/>
-    <link name="${name}">
+  <!-- MOUNT -->
+    <joint name="${prefix}${name}_mount_joint" type="fixed">
+      <xacro:insert_block name="origin" />
+      <parent link="${parent}" />
+      <child link="${prefix}${name}_mount" />
+    </joint>
+    <link name="${prefix}${name}_mount">
       <visual>
-        <origin rpy="0 0 0" xyz="0 0 0"/>
+        <xacro:insert_block name="origin" />
+        <geometry>
+          <mesh filename="package://sick_safetyscanners2/description/meshes/nanoscan3/visual/mount.dae"/>
+        </geometry>
+      </visual>
+    </link>
+  <!-- SENSOR BASE -->
+    <joint name="${prefix}${name}_base_joint" type="fixed">
+      <origin xyz="${base_x} ${base_y} 0"/>
+      <parent link="${prefix}${name}_mount" />
+      <child link="${prefix}${name}_base" />
+    </joint>
+    <link name="${prefix}${name}_base">
+      <origin xyz="${-base_x} ${-base_y} 0"/>
+    </link>
+  <!-- SENSOR FRAME -->
+    <joint name="${name}_joint" type="fixed">
+      <parent link="${prefix}${name}_base" />
+      <child link="${prefix}${name}" />
+      <origin xyz="0 ${sensor_y} ${sensor_z}" rpy="0 0 ${sensor_rot_z}"/>
+    </joint>
+    <link name="${prefix}${name}">
+      <visual>
+        <origin xyz="${-base_x} ${-(sensor_y + base_y)} ${-sensor_z}" rpy="0 0 0" />
         <geometry>
           <mesh filename="package://sick_safetyscanners2/description/meshes/nanoscan3/visual/nanoscan3.dae"/>
@@ -12,14 +46,4 @@
       </visual>
     </link>
-    <joint name="${prefix}base_joint" type="fixed">
-      <xacro:insert_block name="origin" />
-      <parent link="${parent}" />
-      <child link="${prefix}base_link" />
-    </joint>
-    <joint name="${name}_joint" type="fixed">
-      <parent link="${prefix}base_link" />
-      <child link="${name}" />
-      <origin rpy="0 0 0" xyz="0 0 0"/>
-    </joint>
   </xacro:macro>
 </robot>

Commit message: added collision, colored the sensor mesh

File: description/urdf/nanoscan3/nanoscan3_macro.xacro (robot description, xacro)
@@ -23,4 +23,10 @@
           </geometry>
         </visual>
+        <collision>
+          <xacro:insert_block name="origin" />
+          <geometry>
+            <mesh filename="package://sick_safetyscanners2/description/meshes/nanoscan3/collision/mount.dae"/>
+          </geometry>
+        </collision>
       </link>
       <!-- SENSOR BASE when mounted -->
@@ -55,4 +61,10 @@
         </geometry>
       </visual>
+      <collision>
+        <origin xyz="${-base_x} ${-(sensor_y + base_y)} ${-sensor_z}" rpy="0 0 0" />
+        <geometry>
+          <mesh filename="package://sick_safetyscanners2/description/meshes/nanoscan3/collision/nanoscan3.dae"/>
+        </geometry>
+      </collision>
     </link>
   </xacro:macro>

Commit message: structured mesh files to match sick_scan package: https://github.com/SICKAG/sick_scan/tree/master/meshes

File: description/urdf/nanoscan3/nanoscan3_macro.xacro (robot description, xacro)
@@ -23,5 +23,5 @@
           <xacro:insert_block name="origin" />
           <geometry>
-            <mesh filename="package://sick_safetyscanners2/description/meshes/nanoscan3/visual/mount.dae"/>
+            <mesh filename="package://sick_safetyscanners2/description/meshes/MountingKit_2a.dae"/>
           </geometry>
         </visual>
@@ -29,5 +29,5 @@
           <xacro:insert_block name="origin" />
           <geometry>
-            <mesh filename="package://sick_safetyscanners2/description/meshes/nanoscan3/collision/mount.dae"/>
+            <mesh filename="package://sick_safetyscanners2/description/meshes/MountingKit_2a_collision.stl"/>
           </geometry>
         </collision>
@@ -64,5 +64,5 @@
         <origin xyz="${-base_x} ${-(sensor_y + base_y)} ${-sensor_z}" rpy="0 0 0" />
         <geometry>
-          <mesh filename="package://sick_safetyscanners2/description/meshes/nanoscan3/visual/nanoscan3.dae"/>
+          <mesh filename="package://sick_safetyscanners2/description/meshes/NANS3.dae"/>
         </geometry>
       </visual>
@@ -70,5 +70,5 @@
         <origin xyz="${-base_x} ${-(sensor_y + base_y)} ${-sensor_z}" rpy="0 0 0" />
         <geometry>
-          <mesh filename="package://sick_safetyscanners2/description/meshes/nanoscan3/collision/nanoscan3.dae"/>
+          <mesh filename="package://sick_safetyscanners2/description/meshes/NANS3_collision.stl"/>
         </geometry>
       </collision>

Commit message: Enable workin in Gazebo under humble.

File: description/urdf/nanoscan3/nanoscan3_macro.xacro (robot description, xacro)
@@ -37,10 +37,10 @@
         <visual>
           <geometry>
-            <mesh filename="package://sick_safetyscanners2/description/meshes/MountingKit_2a.dae"/>
+            <mesh filename="file://$(find sick_safetyscanners2)/description/meshes/MountingKit_2a.dae"/>
           </geometry>
         </visual>
         <collision>
           <geometry>
-            <mesh filename="package://sick_safetyscanners2/description/meshes/MountingKit_2a_collision.stl"/>
+            <mesh filename="file://$(find sick_safetyscanners2)/description/meshes/MountingKit_2a_collision.stl"/>
           </geometry>
         </collision>
@@ -77,5 +77,5 @@
         <origin xyz="${-base_x} ${-(sensor_y + base_y)} ${-sensor_z}" rpy="0 0 0" />
         <geometry>
-          <mesh filename="package://sick_safetyscanners2/description/meshes/NANS3.dae"/>
+          <mesh filename="file://$(find sick_safetyscanners2)/description/meshes/NANS3.dae"/>
         </geometry>
       </visual>
@@ -83,5 +83,5 @@
         <origin xyz="${-base_x} ${-(sensor_y + base_y)} ${-sensor_z}" rpy="0 0 0" />
         <geometry>
-          <mesh filename="package://sick_safetyscanners2/description/meshes/NANS3_collision.stl"/>
+          <mesh filename="file://$(find sick_safetyscanners2)/description/meshes/NANS3_collision.stl"/>
         </geometry>
       </collision>

Commit message: Add material for correct representation in Gazebo Sim.

File: description/urdf/nanoscan3/nanoscan3_macro.xacro (robot description, xacro)
@@ -39,4 +39,7 @@
             <mesh filename="file://$(find sick_safetyscanners2)/description/meshes/MountingKit_2a.dae"/>
           </geometry>
+          <material name="black">
+            <color rgba="0.0 0.0 0.0 1.0"/>
+          </material>
         </visual>
         <collision>
@@ -79,4 +82,7 @@
           <mesh filename="file://$(find sick_safetyscanners2)/description/meshes/NANS3.dae"/>
         </geometry>
+        <material name="black">
+          <color rgba="0.0 0.0 0.0 1.0"/>
+        </material>
       </visual>
       <collision>

Commit message: Make urdf compatible with gazebo and when accessing remote robot in rviz.

File: description/urdf/nanoscan3/nanoscan3_macro.xacro (robot description, xacro)
@@ -22,6 +22,19 @@
       gaussian_noise:=0.006
       max_beams:=540
+      simulation:=false
       *origin
     ">
+    <xacro:if value="${simulation}">
+      <xacro:property
+        name="file_prefix"
+        value="file://$(find sick_safetyscanners2)"
+        />
+    </xacro:if>
+    <xacro:unless value="${simulation}">
+      <xacro:property
+        name="file_prefix"
+        value="package://sick_safetyscanners2"
+      />
+    </xacro:unless>
     <xacro:if value="${mounting_kit}">
       <!-- MOUNT -->
@@ -37,5 +50,5 @@
         <visual>
           <geometry>
-            <mesh filename="file://$(find sick_safetyscanners2)/description/meshes/MountingKit_2a.dae"/>
+            <mesh filename="${file_prefix}/description/meshes/MountingKit_2a.dae"/>
           </geometry>
           <material name="black">
@@ -45,5 +58,5 @@
         <collision>
           <geometry>
-            <mesh filename="file://$(find sick_safetyscanners2)/description/meshes/MountingKit_2a_collision.stl"/>
+            <mesh filename="${file_prefix}/description/meshes/MountingKit_2a_collision.stl"/>
           </geometry>
         </collision>
@@ -80,5 +93,5 @@
         <origin xyz="${-base_x} ${-(sensor_y + base_y)} ${-sensor_z}" rpy="0 0 0" />
         <geometry>
-          <mesh filename="file://$(find sick_safetyscanners2)/description/meshes/NANS3.dae"/>
+          <mesh filename="${file_prefix}/description/meshes/NANS3.dae"/>
         </geometry>
         <material name="black">
@@ -89,5 +102,5 @@
         <origin xyz="${-base_x} ${-(sensor_y + base_y)} ${-sensor_z}" rpy="0 0 0" />
         <geometry>
-          <mesh filename="file://$(find sick_safetyscanners2)/description/meshes/NANS3_collision.stl"/>
+          <mesh filename="${file_prefix}/description/meshes/NANS3_collision.stl"/>
         </geometry>
       </collision>
